File: PCB/OptolinkDuoBlock/OptolinkDuoBlock.kicad_pcb (KiCad board)
At the start: 2 copper layers, 142.2 x 52.1 mm, 35 parts, among them J1 USB_Serial_Sniffer, J2 USB_Serial_Communication, J3 Optolink, J4 Optolink, Q1 BC547, Q2 BC547, Q3 BC547, Q4 BC547, Q5 BC547, Q6 SFH309

Commit message: add V1.1.0
Parts:
- J1, J2: footprint Connector_PinHeader_2.54mm:PinHeader_1x06_P2.54mm_Vertical -> Connector_PinSocket_2.54mm:PinSocket_1x06_P2.54mm_Vertical
- J4: renamed from J3; footprint Connector_PinHeader_2.54mm:PinHeader_1x03_P2.54mm_Vertical -> Connector_PinSocket_2.54mm:PinSocket_1x03_P2.54mm_Vertical
- moved J3 38.7 mm to (124.5, 53.3), turned to 0 degrees
- moved J4 38.7 mm to (160.0, 68.6), turned to 180 degrees
- moved J2 2.54 mm to (81.3, 58.4)
- renumbered J4 to J3
Connections:
- D6 pad 1: Net-(D6-Pad1) -> Net-(D6-K)
- D6 pad 2: Net-(D6-Pad2) -> Net-(D6-A)
- J3 pad 1: Net-(D6-Pad1) -> Net-(J3-Pin_1)
- J3 pad 2: Net-(D6-Pad2) -> +3V3
- J3 pad 3: Net-(J4-Pad3) -> Net-(J3-Pin_3)
- J4 pad 1: Net-(J3-Pad1) -> Net-(D6-K)
- J4 pad 2: +3V3 -> Net-(D6-A)
- J4 pad 3: Net-(J3-Pad3) -> Net-(J4-Pin_3)
- Q6 pad 1: Net-(D6-Pad2) -> Net-(D6-A)
- Q6 pad 2: Net-(J4-Pad3) -> Net-(J4-Pin_3)
- R5 pad 1: Net-(J3-Pad1) -> Net-(J3-Pin_1)
- R7 pad 1: Net-(J3-Pad3) -> Net-(J3-Pin_3)
Routing:
- net Net-(D6-Pad2): track 25.4 -> 0.00 mm
- net Net-(D6-A): track 0.00 -> 25.4 mm
- net Net-(J4-Pin_3): track 0.00 -> 15.2 mm
- net Net-(J4-Pad3): track 15.2 -> 0.00 mm
- net Net-(J3-Pin_1): track 0.00 -> 12.7 mm
- net Net-(J3-Pad1): track 12.7 -> 0.00 mm
- net Net-(D6-Pad1): track 12.7 -> 0.00 mm
- net Net-(D6-K): track 0.00 -> 12.7 mm
- net Net-(J3-Pin_3): track 0.00 -> 10.2 mm
- net Net-(J3-Pad3): track 10.2 -> 0.00 mm
Other:
- net class Default removed
